File: dual_axis_pv/kicad_version_control/ahmed/dualaxis.kicad_pcb (KiCad board)
At the start: 2 copper layers, 138 x 94.5 mm, 15 parts, among them J1 Conn_01x01, J10 PR_4, J2 Conn_01x01, J3 Conn_01x01, J4 Conn_01x01, J5 Conn_01x01, J6 Conn_01x01, J7 PR_1, J8 PR_2, J9 PR_3

Commit message: added pcb and schematic 11/21
Other:
- board size 138 x 94.5 mm -> 125.5 x 91 mm
Changed lines of the file:
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@@
 	)
 	(gr_rect
-		(start 43 12.5)
-		(end 181 107)
+		(start 39.5 16)
+		(end 165 107)
 		(stroke
 			(width 0.05)
@@
 		(polygon
 			(pts
-				(xy 43 12.5) (xy 181 12.5) (xy 181 107) (xy 43 107)
-			)
-		)
+				(xy 39.5 107) (xy 165 107) (xy 165 16) (xy 39.5 16)
+			)
+		)
